File: Tamagotchi/Tamagotchi.kicad_pcb (KiCad board)
At the start: 2 copper layers, 84.6 x 97.9 mm, 26 parts, among them J1 Battery connector, SW4 SW_Push, SW5 SW_Push, SW6 SW_Push, U3 XIAO-ESP32-C3-SMD, U4 DM-OLED096-636

Commit message: finally figured out battery
Parts:
- removed the REF** at (53.0, 65.5)
- removed the REF** at (75.0, 65.5)
- removed the REF** at (75.0, 87.5)
- removed the REF** at (53.0, 87.5)
- added J1: Battery connector, Connector_PinHeader_2.54mm:PinHeader_1x02_P2.54mm_Vertical, F.Cu at (37.0, 86.0)
- added J2: Programing, Connector_PinHeader_2.54mm:PinHeader_1x04_P2.54mm_Vertical, F.Cu at (82.5, 73.0)
Routing:
- net Net-(J1-Pin_1): track 11.1 -> 17.3 mm
- net GND: track 190.7 -> 196.3 mm
- added copper zone on F.Cu, net GND

Commit message: ...
Parts:
- moved J2 6.50 mm to (89.0, 73.0)
Changed lines of the file:
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@@
 	(footprint "Connector_PinHeader_2.54mm:PinHeader_1x04_P2.54mm_Vertical"
 		(layer "F.Cu")
-		(at 82.5 73)
+		(at 89 73)
 		(descr "Through hole straight pin header, 1x04, 2.54mm pitch, single row")
 		(tags "Through hole pin header THT 1x04 2.54mm single row")
@@
 		)
 		(min_thickness 0.25)
-		(fill
+		(fill yes
 			(thermal_gap 0.5)
 			(thermal_bridge_width 0.5)
